Commit message: .

File: my_robot/urdf/my_robot.gazebo.xacro (robot description, xacro)
@@ -27,5 +27,5 @@
   </gazebo>
   <!-- RGBD Camera -->
-  <gazebo reference="camera_link">
+  <gazebo reference="camera">
     <sensor type="depth" name="camera">
       <always_on>1</always_on>

File: my_robot/urdf/my_robot.urdf.xacro (robot description, xacro)
@@ -153,10 +153,10 @@
   </joint>
   <!-- RBGD Camera link -->
-  <link name="camera_link_optical">
+  <link name="camera_optical">
   </link>
   <!-- RBGD Camera joint -->
   <joint name="camera_optical_joint" type="fixed">
     <origin xyz="0 0 0" rpy="-1.5707 0 -1.5707" />
-    <parent link="camera_link" />
+    <parent link="camera" />
     <child link="camera_link_optical" />
   </joint>

Commit message: .

File: my_robot/urdf/my_robot.gazebo.xacro (robot description, xacro)
@@ -27,6 +27,6 @@
   </gazebo>
   <!-- RGBD Camera -->
-  <gazebo reference="camera">
-    <sensor type="depth" name="camera">
+  <gazebo reference="camera_link">
+    <sensor type="depth" name="camera_1">
       <always_on>1</always_on>
       <update_rate>20.0</update_rate>

File: my_robot/urdf/my_robot.urdf.xacro (robot description, xacro)
@@ -124,5 +124,5 @@
   </joint>
   <!-- Camera link -->
-  <link name="camera">
+  <link name="camera_link">
     <origin xyz="0 0 0" rpy="0 0 0" />
     <inertial>
@@ -148,16 +148,16 @@
   <joint name="camera_joint" type="fixed">
     <parent link="chassis" />
-    <child link="camera" />
+    <child link="camera_link" />
     <origin xyz="0.2 0 0" rpy="0 0 0" />
     <axis xyz="0 1 0" />
   </joint>
   <!-- RBGD Camera link -->
-  <link name="camera_optical">
+  <link name="camera_optical_link">
   </link>
   <!-- RBGD Camera joint -->
   <joint name="camera_optical_joint" type="fixed">
     <origin xyz="0 0 0" rpy="-1.5707 0 -1.5707" />
-    <parent link="camera" />
-    <child link="camera_optical" />
+    <parent link="camera_link" />
+    <child link="camera_optical_link" />
   </joint>
   <!-- Hokuyo LiDAR link -->

Commit message: .

File: my_robot/urdf/my_robot.gazebo.xacro (robot description, xacro)
@@ -27,5 +27,5 @@
   </gazebo>
   <!-- RGBD Camera -->
-  <gazebo reference="camera_link">
+  <gazebo reference="camera">
     <sensor type="depth" name="camera_1">
       <always_on>1</always_on>
@@ -50,5 +50,5 @@
         <updateRate>10.0</updateRate>
         <cameraName>camera</cameraName>
-        <frameName>camera_link_optical</frameName>
+        <frameName>camera_optical</frameName>
         <imageTopicName>rgb/image_raw</imageTopicName>
         <depthImageTopicName>depth/image_raw</depthImageTopicName>

File: my_robot/urdf/my_robot.urdf.xacro (robot description, xacro)
@@ -124,5 +124,5 @@
   </joint>
   <!-- Camera link -->
-  <link name="camera_link">
+  <link name="camera">
     <origin xyz="0 0 0" rpy="0 0 0" />
     <inertial>
@@ -153,11 +153,11 @@
   </joint>
   <!-- RBGD Camera link -->
-  <link name="camera_optical_link">
+  <link name="camera_optical">
   </link>
   <!-- RBGD Camera joint -->
   <joint name="camera_optical_joint" type="fixed">
     <origin xyz="0 0 0" rpy="-1.5707 0 -1.5707" />
-    <parent link="camera_link" />
-    <child link="camera_optical_link" />
+    <parent link="camera" />
+    <child link="camera_optical" />
   </joint>
   <!-- Hokuyo LiDAR link -->
