Commit message: .

File: my_robot/urdf/my_robot.urdf.xacro (robot description, xacro)
@@ -159,5 +159,5 @@
     <origin xyz="0 0 0" rpy="-1.5707 0 -1.5707" />
     <parent link="camera" />
-    <child link="camera_link_optical" />
+    <child link="camera_optical" />
   </joint>
   <!-- Hokuyo LiDAR link -->

Commit message: .

File: my_robot/urdf/my_robot.urdf.xacro (robot description, xacro)
@@ -148,5 +148,5 @@
   <joint name="camera_joint" type="fixed">
     <parent link="chassis" />
-    <child link="camera_link" />
+    <child link="camera" />
     <origin xyz="0.2 0 0" rpy="0 0 0" />
     <axis xyz="0 1 0" />
